File: addon/samd-dev-addon.kicad_pcb (KiCad board)
At the start: 2 copper layers, 30 x 30 mm, 32 parts, among them J1 USB_B_Micro, J2 Conn_01x10, J3 Conn_01x10, SW1 SW_Push, SW2 SW_Push, SW3 SW_Push, U1 MCP1700-3302E_SOT23, U2 FT232RL, U3 Si7020-A20, U4 ADXL343

Commit message: v2.1 manufactured
Parts:
- added U5: MS5607-02BA, Package_LGA:LGA-8_3x5mm_P1.25mm, F.Cu at (123.2, 96.2)
- moved R5 12.4 mm to (106.0, 92.8), turned to 180 degrees
- moved R4 6.02 mm to (106.0, 95.2), turned to 180 degrees
- moved SW3 2.25 mm to (118.8, 96.8)
- moved R3 2.00 mm to (106.0, 97.8), turned to 180 degrees
- moved SW1 0.75 mm to (109.8, 96.8)
- moved SW2 0.75 mm to (114.2, 96.8)
Connections:
- net /PA03 renamed Net-(J3-Pad7)
- net /PA04 renamed Net-(J3-Pad8)
- net /PA30 renamed Net-(J3-Pad2)
- net /PA31 renamed Net-(J3-Pad3)
- net /~RST renamed Net-(J3-Pad1)
- U4 pad 8: Net-(U4-Pad8) -> /PA02
Routing:
- net /PA07: track 16.9 -> 2.84 mm
- net Net-(R5-Pad1): track 6.33 -> 16.0 mm
- net /PA02: track 0.00 -> 8.17 mm, vias 0 -> 1
- net /PA06: track 10.7 -> 2.84 mm
- net Net-(R4-Pad1): track 6.33 -> 11.5 mm
- net /PA22: track 22.0 -> 26.3 mm
- net /PA05: track 6.24 -> 2.86 mm
- net +3V3: track 62.0 -> 64.3 mm
- net /PA23: track 13.5 -> 15.6 mm
- net GND: vias 15 -> 20
